File: IO_Conn.kicad_sch (KiCad schematic)
At the start: 49 parts, among them J1 MJ-3502N, J2 MODEM, J3 PRINTER, J4 External Floppy, J5 MOUSE, J6 FLOPPY_Internal, J9 RJ22, Q2 2N4403, Q3 2N4401, U10B301 4120R-601-250/201LF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

Commit message: Add files via upload
After obtaining actual  128k board, certain component placement tweaks were made. Board was re-routed based on those changes.
Other:
- note added: "NOTE: FB are on the schematic as 27-ohm resistors. Must have been a late design change."
- note added: "NOTE: On the production board, C49/C50 are 1N5234B 6.2v/550mW zener diodes with the anodes to ground...voltage clamps?"
- note added: "NOTE: Production board used packs with the number CRL8425L (which looks like a date) and "115-0002"."
- note removed: "Note: FB are on the schematic as 27-ohm resistors."
Changed lines of the file:
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@@
     (stroke (width 0) (type default) (color 0 0 0 0))
-  )
-  (text "Note: FB are on the schematic as\n27-ohm resistors."
-    (at 289.306 78.486 0)
-    (effects (font (size 1.27 1.27)) (justify left bottom))
   )
   (text "Floppy - Ext/Int" (at 167.386 18.796 0)
     (effects (font (size 2.0066 2.0066) (thickness 0.4013) bold) (justify left bottom))
+  )
+  (text "NOTE: Production board used packs with the\nnumber CRL8425L (which looks like a date)\nand \"115-0002\"."
+    (at 357.886 82.804 0)
+    (effects (font (size 1.27 1.27)) (justify left bottom))
   )
   (text "Modem" (at 39.878 18.034 0)
@@
     (effects (font (size 1.27 1.27)) (justify right bottom))
   )
+  (text "NOTE: FB are on the schematic as\n27-ohm resistors. Must have been\na late design change."
+    (at 288.29 77.978 0)
+    (effects (font (size 1.27 1.27)) (justify left bottom))
+  )
   (text "Glitch filters are on the side of the schematic." (at 47.244 54.102 0)
     (effects (font (size 1.27 1.27)) (justify left bottom))
@@
   (text "NOTE: External floppy connector J4 is \na custom-shell DB19F (10-over-9).\nTE/Tyco/AMP #745971-1 or\nEDC 111468-2"
     (at 216.408 22.86 0)
+    (effects (font (size 1.27 1.27)) (justify left bottom))
+  )
+  (text "NOTE: FB are on the schematic as\n27-ohm resistors. Must have been\na late design change."
+    (at 235.712 198.628 0)
     (effects (font (size 1.27 1.27)) (justify left bottom))
   )
@@
     (effects (font (size 2.0066 2.0066) (thickness 0.4013) bold) (justify left bottom))
   )
+  (text "NOTE: On the production board, C49/C50\nare 1N5234B 6.2v/550mW zener diodes with\nthe anodes to ground...voltage clamps?"
+    (at 242.824 227.838 180)
+    (effects (font (size 1.27 1.27)) (justify right bottom))
+  )
   (label "MS.FY2" (at 278.384 56.134 180)
