File: Power.kicad_sch (KiCad schematic)
At the start: 77 parts, among them J7 Power, Q1 LM7905_TO220, SW2 RESET, U15B201 344-0040, U2B201 15.6672MHz, U4D201 74LS04, U7C201 LM311, Y1 32.768kHz

Commit message: Add files via upload
After obtaining actual  128k board, certain component placement tweaks were made. Board was re-routed based on those changes.
Parts:
- C20, C5: footprint Capacitor_THT:CP_Axial_L11.0mm_D6.0mm_P18.00mm_Horizontal -> Capacitor_THT:CP_Axial_L11.0mm_D5.0mm_P18.00mm_Horizontal
- C21: footprint Capacitor_THT:C_Axial_L5.1mm_D3.1mm_P10.00mm_Horizontal -> Capacitor_THT:C_Axial_L3.8mm_D2.6mm_P7.50mm_Horizontal
- H201, H202, H203, H204, H205, H206, H207, H208: footprint MountingHole:MountingHole_2.7mm_M2.5_Pad -> TestPoint:TestPoint_Plated_Hole_D2.0mm
Changed lines of the file:
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@@
       (effects (font (size 1.27 1.27)) (justify left) hide)
     )
-    (property "Footprint" "MountingHole:MountingHole_2.7mm_M2.5_Pad" (id 2) (at 148.844 170.18 0)
+    (property "Footprint" "TestPoint:TestPoint_Plated_Hole_D2.0mm" (id 2) (at 148.844 170.18 0)
       (effects (font (size 1.27 1.27)) hide)
     )
@@
       (effects (font (size 1.27 1.27)) (justify left) hide)
     )
-    (property "Footprint" "MountingHole:MountingHole_2.7mm_M2.5_Pad" (id 2) (at 131.572 170.18 0)
+    (property "Footprint" "TestPoint:TestPoint_Plated_Hole_D2.0mm" (id 2) (at 131.572 170.18 0)
       (effects (font (size 1.27 1.27)) hide)
     )
@@
       (effects (font (size 1.27 1.27)) (justify left) hide)
     )
-    (property "Footprint" "MountingHole:MountingHole_2.7mm_M2.5_Pad" (id 2) (at 118.618 170.18 0)
+    (property "Footprint" "TestPoint:TestPoint_Plated_Hole_D2.0mm" (id 2) (at 118.618 170.18 0)
       (effects (font (size 1.27 1.27)) hide)
     )
@@
       (effects (font (size 1.27 1.27)) (justify left) hide)
     )
-    (property "Footprint" "MountingHole:MountingHole_2.7mm_M2.5_Pad" (id 2) (at 140.208 170.18 0)
+    (property "Footprint" "TestPoint:TestPoint_Plated_Hole_D2.0mm" (id 2) (at 140.208 170.18 0)
       (effects (font (size 1.27 1.27)) hide)
     )
@@
       (effects (font (size 1.27 1.27)) (justify left) hide)
     )
-    (property "Footprint" "MountingHole:MountingHole_2.7mm_M2.5_Pad" (id 2) (at 144.526 170.18 0)
+    (property "Footprint" "TestPoint:TestPoint_Plated_Hole_D2.0mm" (id 2) (at 144.526 170.18 0)
       (effects (font (size 1.27 1.27)) hide)
     )
@@
       (effects (font (size 1.27 1.27)) (justify left) hide)
     )
-    (property "Footprint" "MountingHole:MountingHole_2.7mm_M2.5_Pad" (id 2) (at 127.254 170.18 0)
+    (property "Footprint" "TestPoint:TestPoint_Plated_Hole_D2.0mm" (id 2) (at 127.254 170.18 0)
       (effects (font (size 1.27 1.27)) hide)
     )
@@
       (effects (font (size 1.27 1.27)) (justify left) hide)
     )
-    (property "Footprint" "MountingHole:MountingHole_2.7mm_M2.5_Pad" (id 2) (at 135.89 170.18 0)
+    (property "Footprint" "TestPoint:TestPoint_Plated_Hole_D2.0mm" (id 2) (at 135.89 170.18 0)
       (effects (font (size 1.27 1.27)) hide)
     )
@@
       (effects (font (size 1.27 1.27)) (justify left))
     )
-    (property "Footprint" "Capacitor_THT:C_Axial_L5.1mm_D3.1mm_P10.00mm_Horizontal" (id 2) (at 50.038 139.7 0)
+    (property "Footprint" "Capacitor_THT:C_Axial_L3.8mm_D2.6mm_P7.50mm_Horizontal" (id 2) (at 50.038 139.7 0)
       (effects (font (size 1.27 1.27)) hide)
     )
@@
       (effects (font (size 1.27 1.27)) (justify left) hide)
     )
-    (property "Footprint" "MountingHole:MountingHole_2.7mm_M2.5_Pad" (id 2) (at 122.936 170.18 0)
+    (property "Footprint" "TestPoint:TestPoint_Plated_Hole_D2.0mm" (id 2) (at 122.936 170.18 0)
       (effects (font (size 1.27 1.27)) hide)
     )
@@
       (effects (font (size 1.27 1.27)) (justify right))
     )
-    (property "Footprint" "Capacitor_THT:CP_Axial_L11.0mm_D6.0mm_P18.00mm_Horizontal" (id 2) (at 176.022 39.878 0)
+    (property "Footprint" "Capacitor_THT:CP_Axial_L11.0mm_D5.0mm_P18.00mm_Horizontal" (id 2) (at 176.022 39.878 0)
       (effects (font (size 1.27 1.27)) hide)
     )
@@
       (effects (font (size 1.27 1.27)) (justify left))
     )
-    (property "Footprint" "Capacitor_THT:CP_Axial_L11.0mm_D6.0mm_P18.00mm_Horizontal" (id 2) (at 59.69 33.02 0)
-      (effects (font (size 1.27 1.27)) hide)
-    )
+    (property "Footprint" "Capacitor_THT:CP_Axial_L11.0mm_D5.0mm_P18.00mm_Horizontal" (id 2) (at 59.69 33.02 0)
+      (effects (font (size 1.27 1.27)) hide)
+    )
